File: PCB/MacroBoard.kicad_pcb (KiCad board)
At the start: 2 copper layers, 185 x 90 mm, 67 parts, among them J1 Pwr, J2 UART, J3 ADC, J4 I2C, J5 B In, J6 Switch, Q1 2N7002, SW0 SW_Push, SW1 SW_Push, SW10 SW_Push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

Commit message: Revision 1.1 (Firmware WIP)
Parts:
- removed Q1: 2N7002, Package_TO_SOT_SMD:SOT-23
- removed R1: 330, Resistor_SMD:R_1206_3216Metric
- removed R2, R3: 10k, Resistor_SMD:R_1206_3216Metric
- added J6: LED, Connector_Pin:Pin_D0.7mm_L6.5mm_W1.8mm_FlatFork, F.Cu at (209.3, 64.2)
- renumbered J6 to J7, SP1 to RV1, SP2 to RV2, SP3 to RV3, SP4 to RV4, SP5 to RV5
Connections:
- L0 pad 1: LED_2 -> 5V
- L0 pad 2: GND -> LED_2
- L0 pad 3: LED_1 -> GND
- L0 pad 4: LED -> LED_1
- L1 pad 1: Net-(L1-DOUT) -> 5V
- L1 pad 2: GND -> Net-(L1-DOUT)
- L1 pad 3: LED_4 -> GND
- L1 pad 4: LED -> LED_4
- L10 pad 1: Net-(L10-DOUT) -> 5V
- L10 pad 2: GND -> Net-(L10-DOUT)
- L10 pad 3: Net-(L10-DIN) -> GND
- L10 pad 4: LED -> Net-(L10-DIN)
- L11 pad 1: Net-(L11-DOUT) -> 5V
- L11 pad 2: GND -> Net-(L11-DOUT)
- L11 pad 3: Net-(L10-DOUT) -> GND
- L11 pad 4: LED -> Net-(L10-DOUT)
- L12 pad 1: LED_3 -> 5V
- L12 pad 2: GND -> LED_3
- L12 pad 3: Net-(L11-DOUT) -> GND
- L12 pad 4: LED -> Net-(L11-DOUT)
- L2 pad 1: Net-(L2-DOUT) -> 5V
- L2 pad 2: GND -> Net-(L2-DOUT)
- L2 pad 3: Net-(L1-DOUT) -> GND
- L2 pad 4: LED -> Net-(L1-DOUT)
- L3 pad 1: Net-(L3-DOUT) -> 5V
- L3 pad 2: GND -> Net-(L3-DOUT)
- L3 pad 3: Net-(L2-DOUT) -> GND
- L3 pad 4: LED -> Net-(L2-DOUT)
- L4 pad 1: unconnected-(L4-DOUT-Pad1) -> 5V
- L4 pad 2: GND -> LED
- L4 pad 3: Net-(L3-DOUT) -> GND
- L4 pad 4: LED -> Net-(L3-DOUT)
- L5 pad 1: Net-(L5-DOUT) -> 5V
- L5 pad 2: GND -> Net-(L5-DOUT)
- L5 pad 3: LED_3 -> GND
- L5 pad 4: LED -> LED_3
- L6 pad 1: Net-(L6-DOUT) -> 5V
- L6 pad 2: GND -> Net-(L6-DOUT)
- L6 pad 3: Net-(L5-DOUT) -> GND
- L6 pad 4: LED -> Net-(L5-DOUT)
- L7 pad 1: Net-(L7-DOUT) -> 5V
- L7 pad 2: GND -> Net-(L7-DOUT)
- L7 pad 3: Net-(L6-DOUT) -> GND
- L7 pad 4: LED -> Net-(L6-DOUT)
- L8 pad 1: LED_4 -> 5V
- L8 pad 2: GND -> LED_4
- L8 pad 3: Net-(L7-DOUT) -> GND
- L8 pad 4: LED -> Net-(L7-DOUT)
- L9 pad 1: Net-(L10-DIN) -> 5V
- L9 pad 2: GND -> Net-(L10-DIN)
- L9 pad 3: LED_2 -> GND
- L9 pad 4: LED -> LED_2
- RPPW1 pad 10: LVL_CON -> unconnected-(RPPW1-GPIO7-Pad10)
- RPPW1 pad 9: unconnected-(RPPW1-GPIO6-Pad9) -> LED_1
Routing:
- net LED: track 425.0 -> 93.6 mm, vias 10 -> 1
- net 5V: track 177.0 -> 427.5 mm, vias 2 -> 14
- net LVL_CON: track 100.1 -> 0.00 mm, vias 3 -> 0
- net LED_1: track 78.7 -> 54.0 mm, vias 4 -> 1
- net Net-(L2-DOUT): track 14.8 -> 0.00 mm, vias 2 -> 0
- net Net-(L3-DOUT): track 14.8 -> 0.00 mm, vias 2 -> 0
- net Net-(L1-DOUT): track 14.6 -> 0.00 mm, vias 2 -> 0
- net 3V3: track 218.8 -> 213.2 mm
- net LED_2: track 46.3 -> 51.6 mm, vias 0 -> 4
- net LED_3: track 93.6 -> 96.2 mm
- net LED_4: track 94.0 -> 96.2 mm
Other:
- board text added: "rev. 1.1"
- board text removed: "rev. 1.0"
