File: PCB/MacroBoard.kicad_sch (KiCad schematic)
At the start: 57 parts, among them J1 Pwr, J2 UART, J3 ADC, J4 I2C, J5 B In, J6 Switch, SW0 SW_Push, SW1 SW_Push, SW10 SW_Push, SW11 SW_Push, SW12 SW_Push, SW2 SW_Push, SW3 SW_Push, SW4 SW_Push, SW5 SW_Push, SW6 SW_Push, SW7 SW_Push, SW8 SW_Push, SW9 SW_Push

Commit message: New LED Footprint, new routings
Parts:
- L0, L1, L10, L11, L12, L2, L3, L4, L5, L6, L7, L8, L9: value SK6812MINI -> SK6812MINI-E; footprint Custom:LED_SK6812MINI_PLCC4_3.5x3.5mm_P1.75mm -> LibraryTool:SK6812MINIE

Commit message: Updated PCB, increased tracks and vias size, added level converter
Parts:
- added C5: 10uF, Capacitor_SMD:C_1206_3216Metric, symbol Device:C
- added C6: 100uF, Capacitor_SMD:C_1206_3216Metric, symbol Device:C
- added Q1: 2N7002, Package_TO_SOT_SMD:SOT-23, symbol Transistor_FET:2N7002
- added R2, R3: 10k, Resistor_SMD:R_1206_3216Metric, symbol Device:R
- RPPW1: footprint Raspberry Pi Pico:MODULE_SC0918 -> RPiP:MODULE_SC0918
Connections:
- net 3V3: now also C5.1, C6.1, Q1.1 (G), R2.2
- net 5V: now also R3.2
- net GND: now also RV1.MP (MountPin), RV2.MP (MountPin), RV3.MP (MountPin), RV4.MP (MountPin), RV5.MP (MountPin), C5.2, C6.2
- net LED_1: now also Q1.3 (D), R3.1; no longer RPPW1.10 (GPIO7)
- new net LVL_CON: Q1.2 (S), R2.1, RPPW1.10 (GPIO7)
Other:
- moved on the sheet: MUX1

Commit message: Revision 1.1 (Firmware WIP)
Parts:
- removed L0, L1, L10, L11, L12, L2, L3, L4, L5, L6, L7, L8, L9: SK6812MINI-E, LibraryTool:SK6812MINIE, symbol LED:SK6812MINI
- removed Q1: 2N7002, Package_TO_SOT_SMD:SOT-23, symbol Transistor_FET:2N7002
- removed R1: 330, Resistor_SMD:R_1206_3216Metric, symbol Device:R
- removed R2, R3: 10k, Resistor_SMD:R_1206_3216Metric, symbol Device:R
- added J6: LED, Connector_Pin:Pin_D0.7mm_L6.5mm_W1.8mm_FlatFork, symbol Connector:Conn_01x01_Socket
- added L0, L1, L10, L11, L12, L2, L3, L4, L5, L6, L7, L8, L9: SK6812MINI-E, LibraryTool:SK6812MINIE, symbol LED:SK6812MINI-E
- renumbered J6 to J7
Connections:
- net 5V: now also L0.1 (VDD), L1.1 (VDD), L10.1 (VDD), L11.1 (VDD), L12.1 (VDD), L2.1 (VDD), L3.1 (VDD), L4.1 (VDD), L5.1 (VDD), L6.1 (VDD), L7.1 (VDD), L8.1 (VDD), L9.1 (VDD)
- net GND: now also L0.3 (GND), L1.3 (GND), L10.3 (GND), L11.3 (GND), L12.3 (GND), L2.3 (GND), L3.3 (GND), L4.3 (GND), L5.3 (GND), L6.3 (GND), L7.3 (GND), L8.3 (GND), L9.3 (GND)
- net LED: now also J6.1 (Pin_1), L4.2 (DOUT)
- net LED_1: now also RPPW1.9 (GPIO6), L0.4 (DIN)
- net LED_2: now also L0.2 (DOUT), L9.4 (DIN)
- net LED_3: now also L12.2 (DOUT), L5.4 (DIN)
- net LED_4: now also L1.4 (DIN), L8.2 (DOUT)
- net LVL_CON: no longer names the net of RPPW1.10 (GPIO7)
- new net: L11.2 (DOUT), L12.4 (DIN)
- new net: L10.2 (DOUT), L11.4 (DIN)
- new net: L2.2 (DOUT), L3.4 (DIN)
- new net: L1.2 (DOUT), L2.4 (DIN)
- new net: L5.2 (DOUT), L6.4 (DIN)
- new net: L10.4 (DIN), L9.2 (DOUT)
- new net: L3.2 (DOUT), L4.4 (DIN)
- new net: L7.2 (DOUT), L8.4 (DIN)
- new net: L6.2 (DOUT), L7.4 (DIN)
Other:
- company: (none) -> Lorenzo Magni
